Commit message: All included

File: urdf/zumoShield.urdf (robot description, URDF)
Before this commit: robot zumo32u4, 1 links, 0 joints
Links:
- link base_link: geometry visual mesh filename=package://cartographer_ros/urdf/zumoShield.STL scale=1 1 1

Commit message: Update zumoShield.urdf

File: urdf/zumoShield.urdf (robot description, URDF)
Before this commit: robot zumoShield, 1 links, 0 joints
Links:
- link base_link: geometry visual mesh filename=package://zumoShield/urdf/zumoShield.STL scale=1 1 1
